Commit message: pp

File: Genesis/goat/goat_rover_2.urdf (robot description, URDF)
Before this commit: robot goat_rover, 23 links, 22 joints
Links:
- link seg_XnYn_Xneg: mass 0.000393 -> 0.008; geometry collision box size=0.2769 0.012 0.012; collision box size=0.2769 0.020 0.020
- link seg_XnYn_Yneg: mass 0.000650 -> 0.015; geometry collision box size=0.4581 0.012 0.012; collision box size=0.4581 0.020 0.020
- link seg_XnYp_Xneg: mass 0.000393 -> 0.008; geometry collision box size=0.2769 0.012 0.012; collision box size=0.2769 0.020 0.020
- link seg_XnYp_Ypos: mass 0.000650 -> 0.015; geometry collision box size=0.4581 0.012 0.012; collision box size=0.4581 0.020 0.020
- link seg_XpYn_Xpos: mass 0.000393 -> 0.008; geometry collision box size=0.2769 0.012 0.012; collision box size=0.2769 0.020 0.020
- link seg_XpYn_Yneg: mass 0.000650 -> 0.015; geometry collision box size=0.4581 0.012 0.012; collision box size=0.4581 0.020 0.020
- link seg_XpYp_Xpos: mass 0.000393 -> 0.008; geometry collision box size=0.2769 0.012 0.012; collision box size=0.2769 0.020 0.020
- link seg_XpYp_Ypos: mass 0.000650 -> 0.015; geometry collision box size=0.4581 0.012 0.012; collision box size=0.4581 0.020 0.020
- link wheel_X_neg: geometry collision cylinder length=0.06 radius=0.05; visual box size=0.25 0.01 0.01
- link wheel_X_pos: geometry collision cylinder length=0.06 radius=0.05; visual box size=0.25 0.01 0.01
- link wheel_Y_neg: geometry collision cylinder length=0.06 radius=0.05; visual box size=0.25 0.01 0.01
- link wheel_Y_pos: geometry collision cylinder length=0.06 radius=0.05; visual box size=0.25 0.01 0.01
Joints:
- joint wheel_joint_X_neg: origin xyz=0.0 -0.05 0.0 rpy=0 0 0 -> xyz=0.0 0.0 0.0 rpy=0 0 0
- joint wheel_joint_X_pos: origin xyz=0.0 0.05 0.0 rpy=0 0 0 -> xyz=0.0 0.0 0.0 rpy=0 0 0
- joint wheel_joint_Y_neg: origin xyz=0.0 -0.05 0.0 rpy=0 0 0 -> xyz=0.0 0.0 0.0 rpy=0 0 0
- joint wheel_joint_Y_pos: origin xyz=0.0 0.05 0.0 rpy=0 0 0 -> xyz=0.0 0.0 0.0 rpy=0 0 0
